Commit message: Basic Controller Working
desired 0.5 m/s actual 0.4 m/s

File: FrostMechanics/five_link_walker.urdf (robot description, URDF)
Before this commit: robot five_link_walker, 5 links, 4 joints
Links:
- removed link torso
- added link Torso, mass 12
Joints:
- joint LeftHip: parent torso -> Torso
- joint RightHip: parent torso -> Torso
